Commit message: run gazebo o home

File: xacro/gazebo_control.xacro (robot description, xacro)
@@ -2,11 +2,12 @@
 <robot xmlns:xacro="http://www.ros.org/wiki/xacro">
     <gazebo>
-        <plugin name="gz_ros2_control::GazeboSimROS2ControlPlugin" filename="gz_ros2_control-system">
-            <!-- Wheel Information     -->
+        <plugin name="gz::sim::systems::DiffDrive"
+                filename="gz-sim-diff-drive-system">
             <left_joint>left_wheel_joint</left_joint>
             <right_joint>right_wheel_joint</right_joint>
-            <wheel_separation>0.3</wheel_separation>
-            <wheel_diameter>0.1</wheel_diameter>
-            <!-- Limit -->
+            <!-- LƯU Ý: dùng wheel_radius, không phải wheel_diameter -->
+            <wheel_separation>0.35</wheel_separation>
+            <wheel_radius>0.05</wheel_radius>
+            <!-- Limits -->
             <max_wheel_torque>200</max_wheel_torque>
             <max_wheel_acceleration>10.0</max_wheel_acceleration>

File: xacro/robot.xacro (robot description, xacro)
@@ -105,3 +105,8 @@
         <origin xyz="0.24 0 0"/>
     </joint>
+    <gazebo reference="caster_wheel">
+        <material>Gazebo/Black</material>
+        <mu1 value="0.001"/>
+        <mu2 value="0.001"/>
+    </gazebo>
 </robot>
